File: hw/sch_pcb/PCRD01.kicad_pcb (KiCad board)
At the start: 2 copper layers, 50.3 x 30 mm, 39 parts, among them J1 JUMP_3X2, J2 JUMP_5X2, J3 CONN1_2, J4 CONN1_2, J5 Out, P1 _, P2 _, P3 _, P4 _, Q1 BF862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

Commit message: add ust identificators
Parts:
- C1, C10, C11, C12, C13, C2, C3, C5, C6, C7, C8, C9, R1, R10, R11, R2, R3, R4, R5, R6, R7, R8, R9: footprint MLAB_R:SMD-0805 -> Mlab_R:SMD-0805

Commit message: clean layout
Routing:
- net GND: track 50.5 -> 2.75 mm, vias 18 -> 17
- net Net-(C4-Pad1): track 25.8 -> 12.7 mm
- net /A: track 14.3 -> 13.3 mm

Commit message: replace PCB capacitor
Parts:
- C4: value 2pF -> 1pF/NP0 251R15S1R0AV4E; footprint Mlab_C:2pF_PCB -> Mlab_R:SMD-0805; moved to B.Cu
- Q1: value BF862 -> 2SK2394-6; footprint MLAB_IO:SOT-23 -> Package_TO_SOT_SMD:SOT-23
- moved C4 5.21 mm to (150.3, 93.0), turned to 90 degrees
- moved Q1 0.09 mm to (154.4, 88.2), turned to -90 degrees
Routing:
- net Net-(C2-Pad1): track 55.9 -> 3.81 mm
- net V-: track 56.0 -> 48.2 mm
- net /A: track 13.3 -> 8.36 mm
- net V+: track 59.2 -> 56.3 mm
- net Net-(C4-Pad1): track 12.7 -> 10.5 mm

Commit message: uklid layoutu
Parts:
- J3: value CONN1_2 -> HEADER_1x03; footprint Hrebinky:CONN_3_2 -> Mlab_Pin_Headers:Straight_1x03; moved to B.Cu
- moved Q1 2.25 mm to (154.4, 86.0)
- moved R12 0.45 mm to (143.8, 90.4)
- moved C4 0.39 mm to (150.3, 93.4)
- moved R4 0.39 mm to (152.5, 93.4)
- turned J3 to -90 degrees
Connections:
- J3 pad 2: /A -> GND
Routing:
- net /A: track 8.36 -> 10.3 mm
- net GND: track 2.75 -> 1.58 mm
- net V-: track 48.2 -> 47.3 mm
- net Net-(C1-Pad1): track 8.55 -> 7.68 mm

Commit message: rename to 01B
Other:
- board text added: "2023"
- board text added: "PCRD01B"
- board text removed: "2015"
- board text removed: "PCRD01A"
Changed lines of the file:
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@@
     (effects (font (size 1.5 1.5) (thickness 0.3)))
   )
-  (gr_text "PCRD01A" (at 165.858 89.8835) (layer "F.SilkS")
+  (gr_text "PCRD01B" (at 165.858 89.8835) (layer "F.SilkS")
     (effects (font (size 1.5 1.5) (thickness 0.3)))
   )
-  (gr_text "2015" (at 148.2685 80.2315) (layer "F.SilkS")
+  (gr_text "2023" (at 148.2685 80.2315) (layer "F.SilkS")
     (effects (font (size 1.5 1.5) (thickness 0.3)))
   )

Commit message: Edit PCB
Parts:
- C1, C10, C11, C12, C13, C15, C2, C3, C4, C5, C6, C7, C8, C9: footprint Mlab_R:SMD-0805 -> Capacitor_SMD:C_0805_2012Metric
- C14: footprint MLAB_R:SMD-0805 -> Capacitor_SMD:C_0805_2012Metric
- J1, J5: footprint Hrebinky:Pin_Header_Straight_2x03 -> Mlab_Pin_Headers:Straight_2x03
- J2: footprint Hrebinky:Pin_Header_Straight_2x05 -> Mlab_Pin_Headers:Straight_2x05
- J4: footprint Hrebinky:Pin_Header_Straight_1x02 -> Mlab_Pin_Headers:Straight_1x02
- R1, R10, R11, R12, R2, R3, R4, R5, R6, R7, R8, R9: footprint Mlab_R:SMD-0805 -> Resistor_SMD:R_0805_2012Metric
- turned J1 to 180 degrees
- turned J2 to -90 degrees
- turned J4 to 180 degrees
- turned J5 to 180 degrees
Connections:
- J1 pad 2: /+Ubias -> GND
- J1 pad 3: GND -> /+Ubias
- J1 pad 4: GND -> /+Ubias
- J1 pad 5: /+Ubias -> GND
- J2 pad 2: V- -> GND
- J2 pad 3: V+ -> V-
- J2 pad 5: GND -> V+
- J2 pad 6: GND -> V+
- J2 pad 8: V+ -> V-
- J2 pad 9: V- -> GND
- J5 pad 2: Net-(C14-Pad2) -> GND
- J5 pad 3: GND -> Net-(C14-Pad2)
- J5 pad 4: GND -> Net-(C14-Pad2)
- J5 pad 5: Net-(C14-Pad2) -> GND
Other:
- rule pad_to_mask_clearance: 0 -> 0.2
