File: hw/sch_pcb/PCRD01.kicad_sch (KiCad schematic)
At the start: 40 parts, among them J1 JUMP_3X2, J2 JUMP_5X2, J3 CONN1_2, J4 CONN1_2, J5 Out, P1 _, P2 _, P3 _, P4 _, Q1 BF862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

Commit message: add sheet-stamp
Other:
- company: (none) -> www.mlab.cz
- title: (none) -> PCRD01A
Changed lines of the file:
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@@
 (kicad_sch (version 20211123) (generator eeschema)
   (paper "A4")
+  (title_block
+    (title "PCRD01A")
+    (rev "01A")
+    (company "www.mlab.cz")
+  )
   (junction (at 88.9 158.75) (diameter 0) (color 0 0 0 0)
   )

Commit message: add ust identificators
Parts:
- C1: ust_id (none) -> 5e3ff8fc1287502a33bad7a3
- C10, C6: ust_id (none) -> 5c70984712875079b91f8b53
- C11: ust_id (none) -> 5c70984712875079b91f8b41
- C12: ust_id (none) -> 5c70984712875079b91f8b42
- C13: ust_id (none) -> 5c70984712875079b91f8b3d
- C14, C8: ust_id (none) -> 5c70984712875079b91f8b4e
- C15: ust_id (none) -> 5c70984712875079b91f8b50
- C2: ust_id (none) -> 5c70984712875079b91f8b31
- C3, C5, C7, C9: ust_id (none) -> 5c70984712875079b91f8b4c
- C4: footprint Mlab_R:SMD-0805 -> (none); now left out of the parts list
- R1, R12, R2: ust_id (none) -> 5c70984612875079b91f8995
- R10: ust_id (none) -> 5c70984612875079b91f8994
- R11, R6: ust_id (none) -> 5c70984612875079b91f899f
- R3, R4: ust_id (none) -> 5c70984712875079b91f8aac
- R5: ust_id (none) -> 5c70984612875079b91f8993
- R7: ust_id (none) -> 5c70984512875079b91f898e
- R8, R9: ust_id (none) -> 5c70984512875079b91f898f
- U1: ust_id (none) -> 5c70984412875079b91f8799
Changed lines of the file:
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@@
       (effects (font (size 0.762 0.762)))
+    )
+    (property "ust_id" "5c70984612875079b91f8995" (id 4) (at 52.07 87.63 0)
+      (effects (font (size 1.27 1.27)) hide)
     )
     (pin "1")
@@
       (effects (font (size 0.762 0.762)))
     )
+    (property "ust_id" "5c70984612875079b91f8995" (id 4) (at 34.29 100.33 0)
+      (effects (font (size 1.27 1.27)) hide)
+    )
     (pin "1")
     (pin "2")
@@
     (property "Datasheet" "" (id 3) (at 63.5 93.98 0)
       (effects (font (size 1.524 1.524)))
+    )
+    (property "ust_id" "5e3ff8fc1287502a33bad7a3" (id 4) (at 63.5 93.98 0)
+      (effects (font (size 1.27 1.27)) hide)
     )
     (pin "1")
@@
     (property "Datasheet" "" (id 3) (at 100.33 102.87 0)
       (effects (font (size 1.524 1.524)))
+    )
+    (property "ust_id" "5c70984412875079b91f8799" (id 4) (at 100.33 102.87 0)
+      (effects (font (size 1.27 1.27)) hide)
     )
     (pin "1")
@@
       (effects (font (size 0.762 0.762)))
     )
+    (property "ust_id" "5c70984712875079b91f8aac" (id 4) (at 97.79 76.2 0)
+      (effects (font (size 1.27 1.27)) hide)
+    )
     (pin "1")
     (pin "2")
   )
   (symbol (lib_id "PCRD01A-rescue:C") (at 96.52 69.85 270) (unit 1)
-    (in_bom yes) (on_board yes)
+    (in_bom no) (on_board yes)
     (property "Reference" "C4" (id 0) (at 99.06 69.85 0)
       (effects (font (size 1.016 1.016)) (justify left))
@@
       (effects (font (size 1.016 1.016)) (justify left))
     )
-    (property "Footprint" "Mlab_R:SMD-0805" (id 2) (at 92.71 70.8152 0)
+    (property "Footprint" "" (id 2) (at 92.71 70.8152 0)
       (effects (font (size 0.762 0.762)) hide)
     )
@@
       (effects (font (size 1.524 1.524)))
     )
+    (property "ust_id" "5c70984712875079b91f8b4e" (id 4) (at 125.73 102.87 0)
+      (effects (font (size 1.27 1.27)) hide)
+    )
     (pin "1")
     (pin "2")
@@
       (effects (font (size 0.762 0.762)))
     )
+    (property "ust_id" "5c70984612875079b91f8993" (id 4) (at 135.89 111.76 0)
+      (effects (font (size 1.27 1.27)) hide)
+    )
     (pin "1")
     (pin "2")
@@
       (effects (font (size 0.762 0.762)))
     )
+    (property "ust_id" "5c70984612875079b91f899f" (id 4) (at 181.61 111.76 0)
+      (effects (font (size 1.27 1.27)) hide)
+    )
     (pin "1")
     (pin "2")
@@
       (effects (font (size 0.762 0.762)))
     )
+    (property "ust_id" "5c70984512875079b91f898e" (id 4) (at 181.61 129.54 0)
+      (effects (font (size 1.27 1.27)) hide)
+    )
     (pin "1")
     (pin "2")
@@
       (effects (font (size 1.524 1.524)))
     )
+    (property "ust_id" "5c70984712875079b91f8b41" (id 4) (at 190.5 111.76 0)
+      (effects (font (size 1.27 1.27)) hide)
+    )
     (pin "1")
     (pin "2")
@@
       (effects (font (size 0.762 0.762)))
     )
+    (property "ust_id" "5c70984512875079b91f898f" (id 4) (at 201.93 105.41 0)
+      (effects (font (size 1.27 1.27)) hide)
+    )
     (pin "1")
     (pin "2")
@@
       (effects (font (size 0.762 0.762)))
     )
+    (property "ust_id" "5c70984512875079b91f898f" (id 4) (at 219.71 105.41 0)
+      (effects (font (size 1.27 1.27)) hide)
+    )
     (pin "1")
     (pin "2")
@@
       (effects (font (size 1.524 1.524)))
     )
+    (property "ust_id" "5c70984712875079b91f8b42" (id 4) (at 210.82 111.76 0)
+      (effects (font (size 1.27 1.27)) hide)
+    )
     (pin "1")
     (pin "2")
@@
       (effects (font (size 1.524 1.524)))
     )
+    (property "ust_id" "5c70984712875079b91f8b3d" (id 4) (at 241.3 82.55 0)
+      (effects (font (size 1.27 1.27)) hide)
+    )
     (pin "1")
     (pin "2")
@@
       (effects (font (size 0.762 0.762)))
     )
+    (property "ust_id" "5c70984612875079b91f8994" (id 4) (at 231.14 76.2 0)
+      (effects (font (size 1.27 1.27)) hide)
+    )
     (pin "1")
     (pin "2")
@@
       (effects (font (size 0.762 0.762)))
     )
+    (property "ust_id" "5c70984712875079b91f8aac" (id 4) (at 80.01 118.11 0)
+      (effects (font (size 1.27 1.27)) hide)
+    )
     (pin "1")
     (pin "2")
@@
       (effects (font (size 1.524 1.524)))
     )
+    (property "ust_id" "5c70984712875079b91f8b31" (id 4) (at 87.63 118.11 0)
+      (effects (font (size 1.27 1.27)) hide)
+    )
     (pin "1")
     (pin "2")
@@
       (effects (font (size 1.524 1.524)))
     )
+    (property "ust_id" "5c70984712875079b91f8b4e" (id 4) (at 262.89 102.87 0)
+      (effects (font (size 1.27 1.27)) hide)
+    )
     (pin "1")
     (pin "2")
@@
     (property "Datasheet" "" (id 3) (at 270.51 110.49 0)
       (effects (font (size 0.762 0.762)))
+    )
+    (property "ust_id" "5c70984612875079b91f899f" (id 4) (at 270.51 110.49 0)
+      (effects (font (size 1.27 1.27)) hide)
     )
     (pin "1")
@@
       (effects (font (size 1.524 1.524)))
     )
+    (property "ust_id" "5c70984712875079b91f8b4c" (id 4) (at 82.55 165.1 0)
+      (effects (font (size 1.27 1.27)) hide)
+    )
     (pin "1")
     (pin "2")
@@
       (effects (font (size 1.524 1.524)))
     )
+    (property "ust_id" "5c70984712875079b91f8b4c" (id 4) (at 88.9 165.1 0)
+      (effects (font (size 1.27 1.27)) hide)
+    )
     (pin "1")
     (pin "2")
@@
       (effects (font (size 1.524 1.524)))
     )
+    (property "ust_id" "5c70984712875079b91f8b4c" (id 4) (at 107.95 165.1 0)
+      (effects (font (size 1.27 1.27)) hide)
+    )
     (pin "1")
     (pin "2")
@@
       (effects (font (size 1.524 1.524)))
     )
+    (property "ust_id" "5c70984712875079b91f8b4c" (id 4) (at 114.3 165.1 0)
+      (effects (font (size 1.27 1.27)) hide)
+    )
     (pin "1")
     (pin "2")
@@
       (effects (font (size 1.524 1.524)))
     )
+    (property "ust_id" "5c70984712875079b91f8b53" (id 4) (at 120.65 165.1 0)
+      (effects (font (size 1.27 1.27)) hide)
+    )
     (pin "1")
     (pin "2")
@@
     (property "Datasheet" "" (id 3) (at 93.98 165.1 0)
       (effects (font (size 1.524 1.524)))
+    )
+    (property "ust_id" "5c70984712875079b91f8b53" (id 4) (at 93.98 165.1 0)
+      (effects (font (size 1.27 1.27)) hide)
     )
     (pin "1")
@@
       (effects (font (size 0.762 0.762)))
     )
+    (property "ust_id" "5c70984612875079b91f8995" (id 4) (at 52.07 100.33 0)
+      (effects (font (size 1.27 1.27)) hide)
+    )
     (pin "1")
     (pin "2")
@@
     (property "Datasheet" "" (id 3) (at 43.18 106.68 0)
       (effects (font (size 1.524 1.524)))
+    )
+    (property "ust_id" "5c70984712875079b91f8b50" (id 4) (at 43.18 106.68 0)
+      (effects (font (size 1.27 1.27)) hide)
     )
     (pin "1")
@@
     )
     (path "/00000000-0000-0000-0000-0000547638f8"
-      (reference "C4") (unit 1) (value "2pF") (footprint "Mlab_R:SMD-0805")
+      (reference "C4") (unit 1) (value "2pF") (footprint "")
     )
     (path "/00000000-0000-0000-0000-00005483ba04"

Commit message: rename id
Parts:
- C1: UST_ID (none) -> 5e3ff8fc1287502a33bad7a3; ust_id 5e3ff8fc1287502a33bad7a3 -> (none)
- C10, C6: UST_ID (none) -> 5c70984712875079b91f8b53; ust_id 5c70984712875079b91f8b53 -> (none)
- C11: UST_ID (none) -> 5c70984712875079b91f8b41; ust_id 5c70984712875079b91f8b41 -> (none)
- C12: UST_ID (none) -> 5c70984712875079b91f8b42; ust_id 5c70984712875079b91f8b42 -> (none)
- C13: UST_ID (none) -> 5c70984712875079b91f8b3d; ust_id 5c70984712875079b91f8b3d -> (none)
- C14, C8: UST_ID (none) -> 5c70984712875079b91f8b4e; ust_id 5c70984712875079b91f8b4e -> (none)
- C15: UST_ID (none) -> 5c70984712875079b91f8b50; ust_id 5c70984712875079b91f8b50 -> (none)
- C2: UST_ID (none) -> 5c70984712875079b91f8b31; ust_id 5c70984712875079b91f8b31 -> (none)
- C3, C5, C7, C9: UST_ID (none) -> 5c70984712875079b91f8b4c; ust_id 5c70984712875079b91f8b4c -> (none)
- R1, R12, R2: UST_ID (none) -> 5c70984612875079b91f8995; ust_id 5c70984612875079b91f8995 -> (none)
- R10: UST_ID (none) -> 5c70984612875079b91f8994; ust_id 5c70984612875079b91f8994 -> (none)
- R11, R6: UST_ID (none) -> 5c70984612875079b91f899f; ust_id 5c70984612875079b91f899f -> (none)
- R3, R4: UST_ID (none) -> 5c70984712875079b91f8aac; ust_id 5c70984712875079b91f8aac -> (none)
- R5: UST_ID (none) -> 5c70984612875079b91f8993; ust_id 5c70984612875079b91f8993 -> (none)
- R7: UST_ID (none) -> 5c70984512875079b91f898e; ust_id 5c70984512875079b91f898e -> (none)
- R8, R9: UST_ID (none) -> 5c70984512875079b91f898f; ust_id 5c70984512875079b91f898f -> (none)
- U1: UST_ID (none) -> 5c70984412875079b91f8799; ust_id 5c70984412875079b91f8799 -> (none)
Changed lines of the file:
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@@
       (effects (font (size 0.762 0.762)))
     )
-    (property "ust_id" "5c70984612875079b91f8995" (id 4) (at 52.07 87.63 0)
+    (property "UST_ID" "5c70984612875079b91f8995" (id 4) (at 52.07 87.63 0)
       (effects (font (size 1.27 1.27)) hide)
     )
@@
       (effects (font (size 0.762 0.762)))
     )
-    (property "ust_id" "5c70984612875079b91f8995" (id 4) (at 34.29 100.33 0)
+    (property "UST_ID" "5c70984612875079b91f8995" (id 4) (at 34.29 100.33 0)
       (effects (font (size 1.27 1.27)) hide)
     )
@@
       (effects (font (size 1.524 1.524)))
     )
-    (property "ust_id" "5e3ff8fc1287502a33bad7a3" (id 4) (at 63.5 93.98 0)
+    (property "UST_ID" "5e3ff8fc1287502a33bad7a3" (id 4) (at 63.5 93.98 0)
       (effects (font (size 1.27 1.27)) hide)
     )
@@
       (effects (font (size 1.524 1.524)))
     )
-    (property "ust_id" "5c70984412875079b91f8799" (id 4) (at 100.33 102.87 0)
+    (property "UST_ID" "5c70984412875079b91f8799" (id 4) (at 100.33 102.87 0)
       (effects (font (size 1.27 1.27)) hide)
     )
@@
       (effects (font (size 0.762 0.762)))
     )
-    (property "ust_id" "5c70984712875079b91f8aac" (id 4) (at 97.79 76.2 0)
+    (property "UST_ID" "5c70984712875079b91f8aac" (id 4) (at 97.79 76.2 0)
       (effects (font (size 1.27 1.27)) hide)
     )
@@
       (effects (font (size 1.524 1.524)))
     )
-    (property "ust_id" "5c70984712875079b91f8b4e" (id 4) (at 125.73 102.87 0)
+    (property "UST_ID" "5c70984712875079b91f8b4e" (id 4) (at 125.73 102.87 0)
       (effects (font (size 1.27 1.27)) hide)
     )
@@
       (effects (font (size 0.762 0.762)))
     )
-    (property "ust_id" "5c70984612875079b91f8993" (id 4) (at 135.89 111.76 0)
+    (property "UST_ID" "5c70984612875079b91f8993" (id 4) (at 135.89 111.76 0)
       (effects (font (size 1.27 1.27)) hide)
     )
@@
       (effects (font (size 0.762 0.762)))
     )
-    (property "ust_id" "5c70984612875079b91f899f" (id 4) (at 181.61 111.76 0)
+    (property "UST_ID" "5c70984612875079b91f899f" (id 4) (at 181.61 111.76 0)
       (effects (font (size 1.27 1.27)) hide)
     )
@@
       (effects (font (size 0.762 0.762)))
     )
-    (property "ust_id" "5c70984512875079b91f898e" (id 4) (at 181.61 129.54 0)
+    (property "UST_ID" "5c70984512875079b91f898e" (id 4) (at 181.61 129.54 0)
       (effects (font (size 1.27 1.27)) hide)
     )
@@
       (effects (font (size 1.524 1.524)))
     )
-    (property "ust_id" "5c70984712875079b91f8b41" (id 4) (at 190.5 111.76 0)
+    (property "UST_ID" "5c70984712875079b91f8b41" (id 4) (at 190.5 111.76 0)
       (effects (font (size 1.27 1.27)) hide)
     )
@@
       (effects (font (size 0.762 0.762)))
     )
-    (property "ust_id" "5c70984512875079b91f898f" (id 4) (at 201.93 105.41 0)
+    (property "UST_ID" "5c70984512875079b91f898f" (id 4) (at 201.93 105.41 0)
       (effects (font (size 1.27 1.27)) hide)
     )
@@
       (effects (font (size 0.762 0.762)))
     )
-    (property "ust_id" "5c70984512875079b91f898f" (id 4) (at 219.71 105.41 0)
+    (property "UST_ID" "5c70984512875079b91f898f" (id 4) (at 219.71 105.41 0)
       (effects (font (size 1.27 1.27)) hide)
     )
@@
       (effects (font (size 1.524 1.524)))
     )
-    (property "ust_id" "5c70984712875079b91f8b42" (id 4) (at 210.82 111.76 0)
+    (property "UST_ID" "5c70984712875079b91f8b42" (id 4) (at 210.82 111.76 0)
       (effects (font (size 1.27 1.27)) hide)
     )
@@
       (effects (font (size 1.524 1.524)))
     )
-    (property "ust_id" "5c70984712875079b91f8b3d" (id 4) (at 241.3 82.55 0)
+    (property "UST_ID" "5c70984712875079b91f8b3d" (id 4) (at 241.3 82.55 0)
       (effects (font (size 1.27 1.27)) hide)
     )
@@
       (effects (font (size 0.762 0.762)))
     )
-    (property "ust_id" "5c70984612875079b91f8994" (id 4) (at 231.14 76.2 0)
+    (property "UST_ID" "5c70984612875079b91f8994" (id 4) (at 231.14 76.2 0)
       (effects (font (size 1.27 1.27)) hide)
     )
@@
       (effects (font (size 0.762 0.762)))
     )
-    (property "ust_id" "5c70984712875079b91f8aac" (id 4) (at 80.01 118.11 0)
+    (property "UST_ID" "5c70984712875079b91f8aac" (id 4) (at 80.01 118.11 0)
       (effects (font (size 1.27 1.27)) hide)
     )
@@
       (effects (font (size 1.524 1.524)))
     )
-    (property "ust_id" "5c70984712875079b91f8b31" (id 4) (at 87.63 118.11 0)
+    (property "UST_ID" "5c70984712875079b91f8b31" (id 4) (at 87.63 118.11 0)
       (effects (font (size 1.27 1.27)) hide)
     )
@@
       (effects (font (size 1.524 1.524)))
     )
-    (property "ust_id" "5c70984712875079b91f8b4e" (id 4) (at 262.89 102.87 0)
+    (property "UST_ID" "5c70984712875079b91f8b4e" (id 4) (at 262.89 102.87 0)
       (effects (font (size 1.27 1.27)) hide)
     )
@@
       (effects (font (size 0.762 0.762)))
     )
-    (property "ust_id" "5c70984612875079b91f899f" (id 4) (at 270.51 110.49 0)
+    (property "UST_ID" "5c70984612875079b91f899f" (id 4) (at 270.51 110.49 0)
       (effects (font (size 1.27 1.27)) hide)
     )
@@
       (effects (font (size 1.524 1.524)))
     )
-    (property "ust_id" "5c70984712875079b91f8b4c" (id 4) (at 82.55 165.1 0)
+    (property "UST_ID" "5c70984712875079b91f8b4c" (id 4) (at 82.55 165.1 0)
       (effects (font (size 1.27 1.27)) hide)
     )
@@
       (effects (font (size 1.524 1.524)))
     )
-    (property "ust_id" "5c70984712875079b91f8b4c" (id 4) (at 88.9 165.1 0)
+    (property "UST_ID" "5c70984712875079b91f8b4c" (id 4) (at 88.9 165.1 0)
       (effects (font (size 1.27 1.27)) hide)
     )
@@
       (effects (font (size 1.524 1.524)))
     )
-    (property "ust_id" "5c70984712875079b91f8b4c" (id 4) (at 107.95 165.1 0)
+    (property "UST_ID" "5c70984712875079b91f8b4c" (id 4) (at 107.95 165.1 0)
       (effects (font (size 1.27 1.27)) hide)
     )
@@
       (effects (font (size 1.524 1.524)))
     )
-    (property "ust_id" "5c70984712875079b91f8b4c" (id 4) (at 114.3 165.1 0)
+    (property "UST_ID" "5c70984712875079b91f8b4c" (id 4) (at 114.3 165.1 0)
       (effects (font (size 1.27 1.27)) hide)
     )
@@
       (effects (font (size 1.524 1.524)))
     )
-    (property "ust_id" "5c70984712875079b91f8b53" (id 4) (at 120.65 165.1 0)
+    (property "UST_ID" "5c70984712875079b91f8b53" (id 4) (at 120.65 165.1 0)
       (effects (font (size 1.27 1.27)) hide)
     )
@@
       (effects (font (size 1.524 1.524)))
     )
-    (property "ust_id" "5c70984712875079b91f8b53" (id 4) (at 93.98 165.1 0)
+    (property "UST_ID" "5c70984712875079b91f8b53" (id 4) (at 93.98 165.1 0)
       (effects (font (size 1.27 1.27)) hide)
     )
@@
       (effects (font (size 0.762 0.762)))
     )
-    (property "ust_id" "5c70984612875079b91f8995" (id 4) (at 52.07 100.33 0)
+    (property "UST_ID" "5c70984612875079b91f8995" (id 4) (at 52.07 100.33 0)
       (effects (font (size 1.27 1.27)) hide)
     )
@@
       (effects (font (size 1.524 1.524)))
     )
-    (property "ust_id" "5c70984712875079b91f8b50" (id 4) (at 43.18 106.68 0)
-      (effects (font (size 1.27 1.27)) hide)
-    )
+    (property "UST_ID" "5c70984712875079b91f8b50" (id 4) (at 43.18 106.68 0)
+      (effects (font (size 1.27 1.27)) hide)
+    )
